File: HW4/PIC32/PIC32.kicad_pcb (KiCad board)
At the start: 2 copper layers, 50 x 50 mm, 23 parts, among them J1 Battery, J2 LEFT, J3 RIGHT, J4 CP2102, SW1 PWR, SW2 MCLR, SW3 USER, U2 AP7381

Commit message: HW5
Parts:
- moved C3 29.1 mm to (136.7, 113.2), turned to 90 degrees
- moved C2 26.4 mm to (133.0, 111.0), turned to 180 degrees
- moved D3 23.1 mm to (113.0, 128.7)
- moved 330 22.2 mm to (118.3, 135.9)
- moved R3 22.2 mm to (109.4, 135.9)
- moved R2 22.1 mm to (113.8, 135.8)
- moved D2 21.3 mm to (108.1, 128.7)
- moved D1 21.2 mm to (118.0, 128.5)
- moved J1 20.5 mm to (115.5, 108.3)
- moved R5 17.8 mm to (149.0, 114.5), turned to 180 degrees
- moved R4 14.2 mm to (148.7, 111.2), turned to 180 degrees
- moved U1 3.59 mm to (123.7, 114.7)
- moved J2 1.02 mm to (103.0, 117.9)
- moved J4 0.09 mm to (102.3, 102.6)

Commit message: kicad_pcb
Parts:
- J4: footprint Connector_PinSocket_2.54mm:PinSocket_1x06_P2.54mm_Vertical -> ME433:AdaFruit Friend
- moved C6 65.6 mm to (122.3, 146.3), turned to 180 degrees
- moved C4 39.9 mm to (140.2, 128.0), turned to 180 degrees
- moved J1 32.4 mm to (147.7, 110.9)
- moved R4 29.9 mm to (141.3, 140.1), turned to -90 degrees
- moved R5 28.2 mm to (137.3, 140.2), turned to -90 degrees
- moved C5 27.0 mm to (137.5, 135.2)
- moved SW1 20.8 mm to (103.0, 106.7), turned to 90 degrees
- moved J4 20.6 mm to (108.8, 122.1)
- moved C1 14.4 mm to (133.9, 111.4), turned to 180 degrees
- moved U2 13.6 mm to (140.4, 111.6)
- moved C3 11.2 mm to (140.1, 123.8), turned to 180 degrees
- moved C2 11.0 mm to (140.1, 119.5)
- moved R2 4.46 mm to (109.4, 135.9)
- moved R3 4.39 mm to (113.8, 135.9)
- moved SW3 3.35 mm to (128.2, 102.4)
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- renumbered U1 to PIC32MX170f256b
Routing:
- net /Vin: track 0.00 -> 118.3 mm, vias 0 -> 2
- net +3.3V: track 0.00 -> 94.7 mm, vias 0 -> 1
- net /MCLR: track 0.00 -> 77.8 mm, vias 0 -> 3
- net Net-(J1-Pin_1): track 0.00 -> 58.9 mm
- net /YELLOW: track 0.00 -> 55.0 mm, vias 0 -> 1
- net /USER: track 0.00 -> 52.4 mm
- net /GREEN: track 0.00 -> 38.6 mm, vias 0 -> 1
- net /B6: track 0.00 -> 35.3 mm, vias 0 -> 2
- net Net-(J4-Pin_4): track 0.00 -> 26.4 mm, vias 0 -> 1
- net /U1RX: track 0.00 -> 26.2 mm, vias 0 -> 1
- net /A3: track 0.00 -> 25.7 mm
- net /B2: track 0.00 -> 24.5 mm
- net /B0: track 0.00 -> 23.8 mm
- net /B1: track 0.00 -> 23.1 mm
- net /A0: track 0.00 -> 23.1 mm
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